Commit message: update piper-pika urdf

File: src/pika_gripper_description/urdf/piper_pika_gripper_description.urdf (robot description, URDF)
Before this commit: robot piper, 11 links, 10 joints
Links:
- link gripper_base: geometry collision mesh filename=package://pika_gripper_description/meshes/gripper_base_link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; visual mesh filename=package://pika_gripper_description/meshes/gripper_base_link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
- link link7: geometry collision mesh filename=package://pika_gripper_description/meshes/gripper_left_link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; visual mesh filename=package://pika_gripper_description/meshes/gripper_left_link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
- link link8: geometry collision mesh filename=package://pika_gripper_description/meshes/gripper_right_lin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; visual mesh filename=package://pika_gripper_description/meshes/gripper_right_lin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
